Commit message: fixed right_wheel orientation

File: zero_description/urdf/zero.urdf.xacro (robot description, xacro)
@@ -11,4 +11,5 @@
     <origin xyz="0 0 0.0862" rpy="0 0 0" />
 </joint>
+<!-- ................................ MOBILE BASE .................................. -->
     <link name="mobile_base">
         <visual>
@@ -189,11 +190,6 @@
         <origin xyz="0 0 0" rpy="0 0 0" />
     </joint>
-    <link name="front_depthcamera">
-        <inertial>
-            <origin xyz="0 0 0" rpy="0 0 0" />
-            <mass value="1e-9" />
-            <inertia ixx="0" ixy="0" ixz="0" iyy="0" iyz="0" izz="0" />
-        </inertial>
-    </link>
+<!-- ................................ FRONT CAMERA .................................. -->
+    <link name="front_depthcamera"/>
     <joint name="front_depthcamera_frame" type="fixed">
         <origin xyz="-9.0288353571388313412e-08 -0.19999916474089063367 0.030885516604367363458"
@@ -203,11 +199,6 @@
         <axis xyz="0 0 0" />
     </joint>
-    <link name="lidar">
-        <inertial>
-            <origin xyz="0 0 0" rpy="0 0 0" />
-            <mass value="1e-9" />
-            <inertia ixx="0" ixy="0" ixz="0" iyy="0" iyz="0" izz="0" />
-        </inertial>
-    </link>
+<!-- ................................ LIDAR .................................. -->
+    <link name="lidar"/>
     <joint name="lidar_frame" type="fixed">
         <origin xyz="-0.00012191376555154009864 -2.8123243064170910799e-05 0.17509999999999997788"
@@ -217,11 +208,6 @@
         <axis xyz="0 0 0" />
     </joint>
-    <link name="back_depthcamera">
-        <inertial>
-            <origin xyz="0 0 0" rpy="0 0 0" />
-            <mass value="1e-9" />
-            <inertia ixx="0" ixy="0" ixz="0" iyy="0" iyz="0" izz="0" />
-        </inertial>
-    </link>
+    <!-- ................................ BACK DEPTH CAMERA .................................. -->
+    <link name="back_depthcamera"/>
     <joint name="back_depthcamera_frame" type="fixed">
         <origin xyz="-9.0288353654655040259e-08 0.19999916474089080021 0.030885516604367439786"
@@ -231,11 +217,6 @@
         <axis xyz="0 0 0" />
     </joint>
-    <link name="imu">
-        <inertial>
-            <origin xyz="0 0 0" rpy="0 0 0" />
-            <mass value="1e-9" />
-            <inertia ixx="0" ixy="0" ixz="0" iyy="0" iyz="0" izz="0" />
-        </inertial>
-    </link>
+    <!-- ................................ IMU .................................. -->
+    <link name="imu"/>
     <joint name="imu_frame" type="fixed">
         <origin xyz="1.2369906293673038927e-07 6.9982771244703201319e-09 0.14380000000000001115"
@@ -245,5 +226,6 @@
         <axis xyz="0 0 0" />
     </joint>
-    <link name="hub_motor_assembly">
+        <!-- ................................ LEFT WHEEL .................................. -->
+    <link name="left_wheel">
         <visual>
             <origin xyz="0 0 0.0068999999999999894751"
@@ -303,10 +285,11 @@
             rpy="-1.570796326794896558 -0 -1.5707963267948970021" />
         <parent link="mobile_base" />
-        <child link="hub_motor_assembly" />
+        <child link="left_wheel" />
         <axis xyz="0 0 1" />
         <limit effort="1" velocity="20" />
         <joint_properties friction="0.0" />
     </joint>
-    <link name="hub_motor_assembly_2">
+            <!-- ................................ RIGHT WHEEL .................................. -->
+    <link name="right_wheel">
         <visual>
             <origin xyz="0 0 0.0069000000000000033529" rpy="-1.570796326794896558 -0 0" />
@@ -365,9 +348,10 @@
             rpy="1.570796326794896558 -0 -1.570796326794896558" />
         <parent link="mobile_base" />
-        <child link="hub_motor_assembly_2" />
-        <axis xyz="0 0 1" />
+        <child link="right_wheel" />
+        <axis xyz="0 0 -1" />
         <limit effort="1" velocity="20" />
         <joint_properties friction="0.0" />
     </joint>
+            <!-- ................................ FRONT CASTER WHEEL  .................................. -->
     <link name="punch">
         <visual>
@@ -439,4 +423,5 @@
         <joint_properties friction="0.0" />
     </joint>
+    <!-- ................................ BACK CASTER WHEEL  .................................. -->
     <link name="punch_2">
         <visual>
@@ -508,4 +493,5 @@
         <joint_properties friction="0.0" />
     </joint>
+    <!-- ................................  PAYLOAD MODULE  .................................. -->
     <link name="payload_module">
         <visual>

Commit message: Replaced stl meshes with dae

File: zero_description/urdf/zero.urdf.xacro (robot description, xacro)
@@ -18,5 +18,5 @@
                 rpy="0 -0 0" />
             <geometry>
-                <mesh filename="package://zero_description/meshes/mobilebase_body.stl" />
+                <mesh filename="package://zero_description/meshes/mobilebase_body.dae" />
             </geometry>
             <material name="mobilebase_body_material">
@@ -29,7 +29,7 @@
                 rpy="-4.6758354725030644238e-16 0.785398163397448279 -3.306314970319521967e-16" />
             <geometry>
-                <mesh filename="package://zero_description/meshes/push_button_-_yellow__list_rekxsjuglcxeoh_yellow.stl" />
-            </geometry>
-            <material name="push_button_-_yellow__list_rekxsjuglcxeoh_yellow_material">
+                <mesh filename="package://zero_description/meshes/push_button_yellow.dae" />
+            </geometry>
+            <material name="push_button_yellow_material">
                 <color
                     rgba="0.70196078431372543882 0.70196078431372543882 0.70196078431372543882 1.0" />
@@ -40,7 +40,7 @@
                 rpy="-4.6758354725030644238e-16 0.785398163397448279 -3.306314970319521967e-16" />
             <geometry>
-                <mesh filename="package://zero_description/meshes/push_button_-_white__list_rekxsjuglcxeoh_white.stl" />
-            </geometry>
-            <material name="push_button_-_white__list_rekxsjuglcxeoh_white_material">
+                <mesh filename="package://zero_description/meshes/push_button_white.dae" />
+            </geometry>
+            <material name="push_button_white_material">
                 <color
                     rgba="0.70196078431372543882 0.70196078431372543882 0.70196078431372543882 1.0" />
@@ -51,5 +51,5 @@
                 rpy="-1.57079632679489678 -0.785398163397448279 1.57079632679489678" />
             <geometry>
-                <mesh filename="package://zero_description/meshes/e_stop.stl" />
+                <mesh filename="package://zero_description/meshes/e_stop.dae" />
             </geometry>
             <material name="e_stop_material">
@@ -61,7 +61,7 @@
                 rpy="-4.6758354725030644238e-16 0.785398163397448279 -3.306314970319521967e-16" />
             <geometry>
-                <mesh filename="package://zero_description/meshes/push_button_-_red__list_rekxsjuglcxeoh_red.stl" />
-            </geometry>
-            <material name="push_button_-_red__list_rekxsjuglcxeoh_red_material">
+                <mesh filename="package://zero_description/meshes/push_button_red.dae" />
+            </geometry>
+            <material name="push_button_red_material">
                 <color
                     rgba="0.70196078431372543882 0.70196078431372543882 0.70196078431372543882 1.0" />
@@ -72,5 +72,5 @@
                 rpy="-1.5707963267948976682 -1.4835298641951801812 1.5707963267948976682" />
             <geometry>
-                <mesh filename="package://zero_description/meshes/antenna.stl" />
+                <mesh filename="package://zero_description/meshes/antenna.dae" />
             </geometry>
             <material name="antenna_material">
@@ -83,5 +83,5 @@
                 rpy="1.570796326794896558 -0 0" />
             <geometry>
-                <mesh filename="package://zero_description/meshes/base.stl" />
+                <mesh filename="package://zero_description/meshes/base.dae" />
             </geometry>
             <material name="base_material">
@@ -94,5 +94,5 @@
                 rpy="-1.570796326794896558 -0 2.6124255799287991292e-16" />
             <geometry>
-                <mesh filename="package://zero_description/meshes/depth_camera.stl" />
+                <mesh filename="package://zero_description/meshes/depth_camera.dae" />
             </geometry>
             <material name="depth_camera_material">
@@ -104,5 +104,5 @@
                 rpy="-1.5707963267948976682 -1.4835298641951801812 1.5707963267948976682" />
             <geometry>
-                <mesh filename="package://zero_description/meshes/antenna.stl" />
+                <mesh filename="package://zero_description/meshes/antenna.dae" />
             </geometry>
             <material name="antenna_material">
@@ -115,7 +115,7 @@
                 rpy="4.6758354725030644238e-16 -0.785398163397448279 -3.306314970319521967e-16" />
             <geometry>
-                <mesh filename="package://zero_description/meshes/push_button_-_red__list_rekxsjuglcxeoh_red.stl" />
-            </geometry>
-            <material name="push_button_-_red__list_rekxsjuglcxeoh_red_material">
+                <mesh filename="package://zero_description/meshes/push_button_red.dae" />
+            </geometry>
+            <material name="push_button_red_material">
                 <color
                     rgba="0.70196078431372543882 0.70196078431372543882 0.70196078431372543882 1.0" />
@@ -126,5 +126,5 @@
                 rpy="0.785398163397448279 1.9048415650792240013e-17 -1.5707963267948970021" />
             <geometry>
-                <mesh filename="package://zero_description/meshes/battery_indicator.stl" />
+                <mesh filename="package://zero_description/meshes/battery_indicator.dae" />
             </geometry>
             <material name="battery_indicator_material">
@@ -137,5 +137,5 @@
                 rpy="1.570796326794896558 -0 0" />
             <geometry>
-                <mesh filename="package://zero_description/meshes/base.stl" />
+                <mesh filename="package://zero_description/meshes/base.dae" />
             </geometry>
             <material name="base_material">
@@ -148,5 +148,5 @@
                 rpy="1.570796326794896558 -0 2.6124255799287991292e-16" />
             <geometry>
-                <mesh filename="package://zero_description/meshes/depth_camera.stl" />
+                <mesh filename="package://zero_description/meshes/depth_camera.dae" />
             </geometry>
             <material name="depth_camera_material">
@@ -158,5 +158,5 @@
                 rpy="1.570796326794896558 -0 0" />
             <geometry>
-                <mesh filename="package://zero_description/meshes/lidar_lower.stl" />
+                <mesh filename="package://zero_description/meshes/lidar_lower.dae" />
             </geometry>
             <material name="lidar_lower_material">
@@ -169,5 +169,5 @@
                 rpy="1.570796326794896558 -0 0" />
             <geometry>
-                <mesh filename="package://zero_description/meshes/lidar_upper.stl" />
+                <mesh filename="package://zero_description/meshes/lidar_upper.dae" />
             </geometry>
             <material name="lidar_upper_material">
@@ -232,5 +232,5 @@
                 rpy="-1.570796326794896558 -1.095640146140279334e-32 0" />
             <geometry>
-                <mesh filename="package://zero_description/meshes/hub_rim_back.stl" />
+                <mesh filename="package://zero_description/meshes/hub_rim_back.dae" />
             </geometry>
             <material name="hub_rim_back_material">
@@ -244,5 +244,5 @@
                 rpy="3.141592653589793116 7.8260293421734858916e-17 2.7052603405912107881" />
             <geometry>
-                <mesh filename="package://zero_description/meshes/hub_rim_face.stl" />
+                <mesh filename="package://zero_description/meshes/hub_rim_face.dae" />
             </geometry>
             <material name="hub_rim_face_material">
@@ -256,5 +256,5 @@
                 rpy="1.570796326794896558 7.8260293421734858916e-17 2.7052603405912107881" />
             <geometry>
-                <mesh filename="package://zero_description/meshes/hub_tire.stl" />
+                <mesh filename="package://zero_description/meshes/hub_tire.dae" />
             </geometry>
             <material name="hub_tire_material">
@@ -268,5 +268,5 @@
                 rpy="1.570796326794896558 7.8260293421734858916e-17 2.7052603405912107881" />
             <geometry>
-                <mesh filename="package://zero_description/meshes/hub_tire.stl" />
+                <mesh filename="package://zero_description/meshes/hub_tire.dae" />
             </geometry>
         </collision>
@@ -295,5 +295,5 @@
             <origin xyz="0 0 0.0069000000000000033529" rpy="-1.570796326794896558 -0 0" />
             <geometry>
-                <mesh filename="package://zero_description/meshes/hub_rim_back.stl" />
+                <mesh filename="package://zero_description/meshes/hub_rim_back.dae" />
             </geometry>
             <material name="hub_rim_back_material">
@@ -307,5 +307,5 @@
                 rpy="3.141592653589793116 -0 2.7052603405912831747" />
             <geometry>
-                <mesh filename="package://zero_description/meshes/hub_rim_face.stl" />
+                <mesh filename="package://zero_description/meshes/hub_rim_face.dae" />
             </geometry>
             <material name="hub_rim_face_material">
@@ -319,5 +319,5 @@
                 rpy="1.570796326794896558 -0 2.7052603405912831747" />
             <geometry>
-                <mesh filename="package://zero_description/meshes/hub_tire.stl" />
+                <mesh filename="package://zero_description/meshes/hub_tire.dae" />
             </geometry>
             <material name="hub_tire_material">
@@ -331,5 +331,5 @@
                 rpy="1.570796326794896558 -0 2.7052603405912831747" />
             <geometry>
-                <mesh filename="package://zero_description/meshes/hub_tire.stl" />
+                <mesh filename="package://zero_description/meshes/hub_tire.dae" />
             </geometry>
         </collision>
@@ -359,5 +359,5 @@
                 rpy="-1.570796326794896558 -0 0" />
             <geometry>
-                <mesh filename="package://zero_description/meshes/punch.stl" />
+                <mesh filename="package://zero_description/meshes/punch.dae" />
             </geometry>
             <material name="punch_material">
@@ -381,5 +381,5 @@
                 rpy="3.141592653589793116 -0 0" />
             <geometry>
-                <mesh filename="package://zero_description/meshes/tire.stl" />
+                <mesh filename="package://zero_description/meshes/tire.dae" />
             </geometry>
             <material name="tire_material">
@@ -392,5 +392,5 @@
                 rpy="3.141592653589793116 -0 0" />
             <geometry>
-                <mesh filename="package://zero_description/meshes/tire.stl" />
+                <mesh filename="package://zero_description/meshes/tire.dae" />
             </geometry>
         </collision>
@@ -429,5 +429,5 @@
                 rpy="-1.570796326794896558 -0 0" />
             <geometry>
-                <mesh filename="package://zero_description/meshes/punch.stl" />
+                <mesh filename="package://zero_description/meshes/punch.dae" />
             </geometry>
             <material name="punch_material">
@@ -451,5 +451,5 @@
                 rpy="3.141592653589793116 -0 0" />
             <geometry>
-                <mesh filename="package://zero_description/meshes/tire.stl" />
+                <mesh filename="package://zero_description/meshes/tire.dae" />
             </geometry>
             <material name="tire_material">
@@ -462,5 +462,5 @@
                 rpy="3.141592653589793116 -0 0" />
             <geometry>
-                <mesh filename="package://zero_description/meshes/tire.stl" />
+                <mesh filename="package://zero_description/meshes/tire.dae" />
             </geometry>
         </collision>
@@ -500,5 +500,5 @@
                 rpy="-1.6653345369377353037e-16 2.3453346881756870093e-17 6.0540737700961713084e-16" />
             <geometry>
-                <mesh filename="package://zero_description/meshes/standoff2.stl" />
+                <mesh filename="package://zero_description/meshes/standoff2.dae" />
             </geometry>
             <material name="standoff2_material">
@@ -511,5 +511,5 @@
                 rpy="-1.6653345369377353037e-16 2.3453346881756870093e-17 6.0540737700961713084e-16" />
             <geometry>
-                <mesh filename="package://zero_description/meshes/standoff2.stl" />
+                <mesh filename="package://zero_description/meshes/standoff2.dae" />
             </geometry>
         </collision>
@@ -517,5 +517,5 @@
             <origin xyz="-1.9645968037643526314e-08 2.2406632246638525398e-07 -0.25" rpy="0 -0 0" />
             <geometry>
-                <mesh filename="package://zero_description/meshes/payload_system.stl" />
+                <mesh filename="package://zero_description/meshes/payload_system.dae" />
             </geometry>
             <material name="payload_system_material">
@@ -593,5 +593,5 @@
                 rpy="-1.6653345369377353037e-16 2.3453346881756870093e-17 6.0540737700961713084e-16" />
             <geometry>
-                <mesh filename="package://zero_description/meshes/tray.stl" />
+                <mesh filename="package://zero_description/meshes/tray.dae" />
             </geometry>
             <material name="tray_material">
@@ -605,5 +605,5 @@
                 rpy="-1.6653345369377353037e-16 2.3453346881756870093e-17 6.0540737700961713084e-16" />
             <geometry>
-                <mesh filename="package://zero_description/meshes/standoff4.stl" />
+                <mesh filename="package://zero_description/meshes/standoff4.dae" />
             </geometry>
             <material name="standoff4_material">
@@ -616,13 +616,13 @@
                 rpy="-1.6653345369377353037e-16 2.3453346881756870093e-17 6.0540737700961713084e-16" />
             <geometry>
-                <mesh filename="package://zero_description/meshes/standoff4.stl" />
-            </geometry>
-        </collision>
-        <visual>
-            <origin
-                xyz="-1.9645968147830495471e-08 2.2406632255051934257e-07 -0.25000000000000022204"
-                rpy="-1.6653345369377353037e-16 2.3453346881756870093e-17 6.0540737700961713084e-16" />
-            <geometry>
-                <mesh filename="package://zero_description/meshes/standoff1.stl" />
+                <mesh filename="package://zero_description/meshes/standoff4.dae" />
+            </geometry>
+        </collision>
+        <visual>
+            <origin
+                xyz="-1.9645968147830495471e-08 2.2406632255051934257e-07 -0.25000000000000022204"
+                rpy="-1.6653345369377353037e-16 2.3453346881756870093e-17 6.0540737700961713084e-16" />
+            <geometry>
+                <mesh filename="package://zero_description/meshes/standoff1.dae" />
             </geometry>
             <material name="standoff1_material">
@@ -635,5 +635,5 @@
                 rpy="-1.6653345369377353037e-16 2.3453346881756870093e-17 6.0540737700961713084e-16" />
             <geometry>
-                <mesh filename="package://zero_description/meshes/standoff1.stl" />
+                <mesh filename="package://zero_description/meshes/standoff1.dae" />
             </geometry>
         </collision>
@@ -642,5 +642,5 @@
                 rpy="1.1344640137963146742 -0 5.5511151231257836882e-16" />
             <geometry>
-                <mesh filename="package://zero_description/meshes/display.stl" />
+                <mesh filename="package://zero_description/meshes/display.dae" />
             </geometry>
             <material name="display_material">
@@ -654,5 +654,5 @@
                 rpy="-1.6653345369377353037e-16 2.3453346881756870093e-17 6.0540737700961713084e-16" />
             <geometry>
-                <mesh filename="package://zero_description/meshes/standoff3.stl" />
+                <mesh filename="package://zero_description/meshes/standoff3.dae" />
             </geometry>
             <material name="standoff3_material">
@@ -665,5 +665,5 @@
                 rpy="-1.6653345369377353037e-16 2.3453346881756870093e-17 6.0540737700961713084e-16" />
             <geometry>
-                <mesh filename="package://zero_description/meshes/standoff3.stl" />
+                <mesh filename="package://zero_description/meshes/standoff3.dae" />
             </geometry>
         </collision>
