Commit message: Removed material tags

File: zero_description/urdf/zero.urdf.xacro (robot description, xacro)
@@ -20,8 +20,4 @@
                 <mesh filename="package://zero_description/meshes/mobilebase_body.dae" />
             </geometry>
-            <material name="mobilebase_body_material">
-                <color
-                    rgba="0.91764705882352937127 0.91764705882352937127 0.91764705882352937127 1.0" />
-            </material>
         </visual>
         <visual>
@@ -31,8 +27,4 @@
                 <mesh filename="package://zero_description/meshes/push_button_yellow.dae" />
             </geometry>
-            <material name="push_button_yellow_material">
-                <color
-                    rgba="0.70196078431372543882 0.70196078431372543882 0.70196078431372543882 1.0" />
-            </material>
         </visual>
         <visual>
@@ -42,8 +34,4 @@
                 <mesh filename="package://zero_description/meshes/push_button_white.dae" />
             </geometry>
-            <material name="push_button_white_material">
-                <color
-                    rgba="0.70196078431372543882 0.70196078431372543882 0.70196078431372543882 1.0" />
-            </material>
         </visual>
         <visual>
@@ -53,7 +41,4 @@
                 <mesh filename="package://zero_description/meshes/e_stop.dae" />
             </geometry>
-            <material name="e_stop_material">
-                <color rgba="1 0 0 1.0" />
-            </material>
         </visual>
         <visual>
@@ -63,8 +48,4 @@
                 <mesh filename="package://zero_description/meshes/push_button_red.dae" />
             </geometry>
-            <material name="push_button_red_material">
-                <color
-                    rgba="0.70196078431372543882 0.70196078431372543882 0.70196078431372543882 1.0" />
-            </material>
         </visual>
         <visual>
@@ -74,8 +55,4 @@
                 <mesh filename="package://zero_description/meshes/antenna.dae" />
             </geometry>
-            <material name="antenna_material">
-                <color
-                    rgba="0.91764705882352937127 0.91764705882352937127 0.91764705882352937127 1.0" />
-            </material>
         </visual>
         <visual>
@@ -85,8 +62,4 @@
                 <mesh filename="package://zero_description/meshes/base.dae" />
             </geometry>
-            <material name="base_material">
-                <color
-                    rgba="0.98039215686274505668 0.71372549019607844922 0.0039215686274509803377 1.0" />
-            </material>
         </visual>
         <visual>
@@ -96,7 +69,4 @@
                 <mesh filename="package://zero_description/meshes/depth_camera.dae" />
             </geometry>
-            <material name="depth_camera_material">
-                <color rgba="0.86666666666666669627 0.90980392156862743835 1 1.0" />
-            </material>
         </visual>
         <visual>
@@ -106,8 +76,4 @@
                 <mesh filename="package://zero_description/meshes/antenna.dae" />
             </geometry>
-            <material name="antenna_material">
-                <color
-                    rgba="0.91764705882352937127 0.91764705882352937127 0.91764705882352937127 1.0" />
-            </material>
         </visual>
         <visual>
@@ -117,8 +83,4 @@
                 <mesh filename="package://zero_description/meshes/push_button_red.dae" />
             </geometry>
-            <material name="push_button_red_material">
-                <color
-                    rgba="0.70196078431372543882 0.70196078431372543882 0.70196078431372543882 1.0" />
-            </material>
         </visual>
         <visual>
@@ -128,8 +90,4 @@
                 <mesh filename="package://zero_description/meshes/battery_indicator.dae" />
             </geometry>
-            <material name="battery_indicator_material">
-                <color
-                    rgba="0.97254901960784312376 0.52941176470588235947 0.0039215686274509803377 1.0" />
-            </material>
         </visual>
         <visual>
@@ -139,8 +97,4 @@
                 <mesh filename="package://zero_description/meshes/base.dae" />
             </geometry>
-            <material name="base_material">
-                <color
-                    rgba="0.98039215686274505668 0.71372549019607844922 0.0039215686274509803377 1.0" />
-            </material>
         </visual>
         <visual>
@@ -150,7 +104,4 @@
                 <mesh filename="package://zero_description/meshes/depth_camera.dae" />
             </geometry>
-            <material name="depth_camera_material">
-                <color rgba="0.86666666666666669627 0.90980392156862743835 1 1.0" />
-            </material>
         </visual>
         <visual>
@@ -160,8 +111,4 @@
                 <mesh filename="package://zero_description/meshes/lidar_lower.dae" />
             </geometry>
-            <material name="lidar_lower_material">
-                <color
-                    rgba="0.49803921568627451677 0.49803921568627451677 0.49803921568627451677 1.0" />
-            </material>
         </visual>
         <visual>
@@ -171,13 +118,9 @@
                 <mesh filename="package://zero_description/meshes/lidar_upper.dae" />
             </geometry>
-            <material name="lidar_upper_material">
-                <color
-                    rgba="0.88235294117647056211 0.57254901960784310155 0.47843137254901962896 1.0" />
-            </material>
         </visual>
         <inertial>
             <origin xyz="0.0025832041792662259645 0.00025148635105191804182 0.047819657753682694168"
                 rpy="0 0 0" />
-            <mass value="7.8674685914887625415" />
+            <mass value="15.8674685914887625415" />
             <inertia ixx="0.18329434197773372683" ixy="-0.00043336984297835835908"
                 ixz="-0.0015567268215315103845" iyy="0.18539574725265989263"
@@ -234,8 +177,4 @@
                 <mesh filename="package://zero_description/meshes/hub_rim_back.dae" />
             </geometry>
-            <material name="hub_rim_back_material">
-                <color
-                    rgba="0.97254901960784312376 0.52941176470588235947 0.0039215686274509803377 1.0" />
-            </material>
         </visual>
         <visual>
@@ -246,8 +185,4 @@
                 <mesh filename="package://zero_description/meshes/hub_rim_face.dae" />
             </geometry>
-            <material name="hub_rim_face_material">
-                <color
-                    rgba="0.91764705882352937127 0.91764705882352937127 0.91764705882352937127 1.0" />
-            </material>
         </visual>
         <visual>
@@ -258,8 +193,4 @@
                 <mesh filename="package://zero_description/meshes/hub_tire.dae" />
             </geometry>
-            <material name="hub_tire_material">
-                <color
-                    rgba="0.64705882352941179736 0.64705882352941179736 0.64705882352941179736 1.0" />
-            </material>
         </visual>
         <collision>
@@ -297,8 +228,4 @@
                 <mesh filename="package://zero_description/meshes/hub_rim_back.dae" />
             </geometry>
-            <material name="hub_rim_back_material">
-                <color
-                    rgba="0.97254901960784312376 0.52941176470588235947 0.0039215686274509803377 1.0" />
-            </material>
         </visual>
         <visual>
@@ -309,8 +236,4 @@
                 <mesh filename="package://zero_description/meshes/hub_rim_face.dae" />
             </geometry>
-            <material name="hub_rim_face_material">
-                <color
-                    rgba="0.91764705882352937127 0.91764705882352937127 0.91764705882352937127 1.0" />
-            </material>
         </visual>
         <visual>
@@ -321,8 +244,4 @@
                 <mesh filename="package://zero_description/meshes/hub_tire.dae" />
             </geometry>
-            <material name="hub_tire_material">
-                <color
-                    rgba="0.64705882352941179736 0.64705882352941179736 0.64705882352941179736 1.0" />
-            </material>
         </visual>
         <collision>
@@ -361,8 +280,4 @@
                 <mesh filename="package://zero_description/meshes/punch.dae" />
             </geometry>
-            <material name="punch_material">
-                <color
-                    rgba="0.91764705882352937127 0.91764705882352937127 0.91764705882352937127 1.0" />
-            </material>
         </visual>
         <inertial>
@@ -383,8 +298,4 @@
                 <mesh filename="package://zero_description/meshes/tire.dae" />
             </geometry>
-            <material name="tire_material">
-                <color
-                    rgba="0.49803921568627451677 0.49803921568627451677 0.49803921568627451677 1.0" />
-            </material>
         </visual>
         <collision>
@@ -431,8 +342,4 @@
                 <mesh filename="package://zero_description/meshes/punch.dae" />
             </geometry>
-            <material name="punch_material">
-                <color
-                    rgba="0.91764705882352937127 0.91764705882352937127 0.91764705882352937127 1.0" />
-            </material>
         </visual>
         <inertial>
@@ -453,8 +360,4 @@
                 <mesh filename="package://zero_description/meshes/tire.dae" />
             </geometry>
-            <material name="tire_material">
-                <color
-                    rgba="0.49803921568627451677 0.49803921568627451677 0.49803921568627451677 1.0" />
-            </material>
         </visual>
         <collision>
@@ -502,7 +405,4 @@
                 <mesh filename="package://zero_description/meshes/standoff2.dae" />
             </geometry>
-            <material name="standoff2_material">
-                <color rgba="0 0 0 1.0" />
-            </material>
         </visual>
         <collision>
@@ -519,8 +419,4 @@
                 <mesh filename="package://zero_description/meshes/payload_system.dae" />
             </geometry>
-            <material name="payload_system_material">
-                <color
-                    rgba="0.91764705882352937127 0.91764705882352937127 0.91764705882352937127 1.0" />
-            </material>
         </visual>
         <!-- Shapes for payload_system -->
@@ -595,8 +491,4 @@
                 <mesh filename="package://zero_description/meshes/tray.dae" />
             </geometry>
-            <material name="tray_material">
-                <color
-                    rgba="0.37254901960784314596 0.38039215686274507888 0.38039215686274507888 1.0" />
-            </material>
         </visual>
         <visual>
@@ -607,7 +499,4 @@
                 <mesh filename="package://zero_description/meshes/standoff4.dae" />
             </geometry>
-            <material name="standoff4_material">
-                <color rgba="0 0 0 1.0" />
-            </material>
         </visual>
         <collision>
@@ -626,7 +515,4 @@
                 <mesh filename="package://zero_description/meshes/standoff1.dae" />
             </geometry>
-            <material name="standoff1_material">
-                <color rgba="0 0 0 1.0" />
-            </material>
         </visual>
         <collision>
@@ -644,8 +530,4 @@
                 <mesh filename="package://zero_description/meshes/display.dae" />
             </geometry>
-            <material name="display_material">
-                <color
-                    rgba="0.56470588235294116863 0.56470588235294116863 0.56470588235294116863 1.0" />
-            </material>
         </visual>
         <visual>
@@ -656,7 +538,4 @@
                 <mesh filename="package://zero_description/meshes/standoff3.dae" />
             </geometry>
-            <material name="standoff3_material">
-                <color rgba="0 0 0 1.0" />
-            </material>
         </visual>
         <collision>
@@ -671,5 +550,5 @@
             <origin xyz="-3.7495602146508909822e-06 0.017289307058686011198 0.59395703720064196851"
                 rpy="0 0 0" />
-            <mass value="17.00660133760975512" />
+            <mass value="5.00660133760975512" />
             <inertia ixx="1.7825536787310567455" ixy="-1.1653610391053570395e-05"
                 ixz="9.2066691289708658952e-06" iyy="1.8011830810656086488"
