Commit message: Optimized URDF

File: zero_description/urdf/zero.urdf.xacro (robot description, xacro)
@@ -18,103 +18,5 @@
                 rpy="0 -0 0" />
             <geometry>
-                <mesh filename="package://zero_description/meshes/mobilebase_body.dae" />
-            </geometry>
-        </visual>
-        <visual>
-            <origin xyz="0.18558108475551546301 0.050000000000000092981 0.12821891524448453259"
-                rpy="-4.6758354725030644238e-16 0.785398163397448279 -3.306314970319521967e-16" />
-            <geometry>
-                <mesh filename="package://zero_description/meshes/push_button_yellow.dae" />
-            </geometry>
-        </visual>
-        <visual>
-            <origin xyz="0.18558108475551543526 1.1102230246251565404e-16 0.12821891524448456035"
-                rpy="-4.6758354725030644238e-16 0.785398163397448279 -3.306314970319521967e-16" />
-            <geometry>
-                <mesh filename="package://zero_description/meshes/push_button_white.dae" />
-            </geometry>
-        </visual>
-        <visual>
-            <origin xyz="0.050580550725237344301 0.18540117237123723837 0.12839882762876278499"
-                rpy="-1.57079632679489678 -0.785398163397448279 1.57079632679489678" />
-            <geometry>
-                <mesh filename="package://zero_description/meshes/e_stop.dae" />
-            </geometry>
-        </visual>
-        <visual>
-            <origin xyz="0.1855810847555154075 -0.04999999999999991257 0.12821891524448456035"
-                rpy="-4.6758354725030644238e-16 0.785398163397448279 -3.306314970319521967e-16" />
-            <geometry>
-                <mesh filename="package://zero_description/meshes/push_button_red.dae" />
-            </geometry>
-        </visual>
-        <visual>
-            <origin xyz="-0.050013022320990196956 0.17818181985266631773 -0.010416397568953073005"
-                rpy="-1.5707963267948976682 -1.4835298641951801812 1.5707963267948976682" />
-            <geometry>
-                <mesh filename="package://zero_description/meshes/antenna.dae" />
-            </geometry>
-        </visual>
-        <visual>
-            <origin xyz="2.2389104848756850518e-17 -0.14500000000000007327 -0.044199999999999996236"
-                rpy="1.570796326794896558 -0 0" />
-            <geometry>
-                <mesh filename="package://zero_description/meshes/base.dae" />
-            </geometry>
-        </visual>
-        <visual>
-            <origin xyz="0.00037417506994241733764 0.17799916474089080842 0.030885528513773852222"
-                rpy="-1.570796326794896558 -0 2.6124255799287991292e-16" />
-            <geometry>
-                <mesh filename="package://zero_description/meshes/depth_camera.dae" />
-            </geometry>
-        </visual>
-        <visual>
-            <origin xyz="-0.07001302232099021472 0.17818181985266626222 -0.010416397568953184027"
-                rpy="-1.5707963267948976682 -1.4835298641951801812 1.5707963267948976682" />
-            <geometry>
-                <mesh filename="package://zero_description/meshes/antenna.dae" />
-            </geometry>
-        </visual>
-        <visual>
-            <origin xyz="-0.18558108475551546301 -0.050000000000000030531 0.12821891524448453259"
-                rpy="4.6758354725030644238e-16 -0.785398163397448279 -3.306314970319521967e-16" />
-            <geometry>
-                <mesh filename="package://zero_description/meshes/push_button_red.dae" />
-            </geometry>
-        </visual>
-        <visual>
-            <origin xyz="-0.1888691312880329265 0.07064999999999996283 0.10796030596349000252"
-                rpy="0.785398163397448279 1.9048415650792240013e-17 -1.5707963267948970021" />
-            <geometry>
-                <mesh filename="package://zero_description/meshes/battery_indicator.dae" />
-            </geometry>
-        </visual>
-        <visual>
-            <origin xyz="-9.5525017435414730954e-17 0.14500000000000001776 -0.044199999999999996236"
-                rpy="1.570796326794896558 -0 0" />
-            <geometry>
-                <mesh filename="package://zero_description/meshes/base.dae" />
-            </geometry>
-        </visual>
-        <visual>
-            <origin xyz="0.00037417506994250060437 -0.17799916474089066964 0.030885504694960957961"
-                rpy="1.570796326794896558 -0 2.6124255799287991292e-16" />
-            <geometry>
-                <mesh filename="package://zero_description/meshes/depth_camera.dae" />
-            </geometry>
-        </visual>
-        <visual>
-            <origin xyz="1.2369906294378053566e-07 6.9982771141252420493e-09 0.14380000000000001115"
-                rpy="1.570796326794896558 -0 0" />
-            <geometry>
-                <mesh filename="package://zero_description/meshes/lidar_lower.dae" />
-            </geometry>
-        </visual>
-        <visual>
-            <origin xyz="1.2369906294378053566e-07 6.9982771141252420493e-09 0.14380000000000001115"
-                rpy="1.570796326794896558 -0 0" />
-            <geometry>
-                <mesh filename="package://zero_description/meshes/lidar_upper.dae" />
+                <mesh filename="package://zero_description/meshes/zero_mobile_base.dae" />
             </geometry>
         </visual>
@@ -172,24 +74,9 @@
     <link name="left_wheel">
         <visual>
-            <origin xyz="0 0 0.0068999999999999894751"
-                rpy="-1.570796326794896558 -1.095640146140279334e-32 0" />
-            <geometry>
-                <mesh filename="package://zero_description/meshes/hub_rim_back.dae" />
-            </geometry>
-        </visual>
-        <visual>
-            <origin
-                xyz="1.1891665430141531362e-14 -2.0816681711721685133e-16 0.062200000000000005285"
-                rpy="3.141592653589793116 7.8260293421734858916e-17 2.7052603405912107881" />
-            <geometry>
-                <mesh filename="package://zero_description/meshes/hub_rim_face.dae" />
-            </geometry>
-        </visual>
-        <visual>
             <origin
                 xyz="1.1911660546815028402e-14 -2.0816681711721685133e-16 0.027249999999999940936"
                 rpy="1.570796326794896558 7.8260293421734858916e-17 2.7052603405912107881" />
             <geometry>
-                <mesh filename="package://zero_description/meshes/hub_tire.dae" />
+                <mesh filename="package://zero_description/meshes/hub_wheel.dae" />
             </geometry>
         </visual>
@@ -199,5 +86,5 @@
                 rpy="1.570796326794896558 7.8260293421734858916e-17 2.7052603405912107881" />
             <geometry>
-                <mesh filename="package://zero_description/meshes/hub_tire.dae" />
+                <mesh filename="package://zero_description/meshes/hub_wheel.dae" />
             </geometry>
         </collision>
@@ -224,23 +111,9 @@
     <link name="right_wheel">
         <visual>
-            <origin xyz="0 0 0.0069000000000000033529" rpy="-1.570796326794896558 -0 0" />
-            <geometry>
-                <mesh filename="package://zero_description/meshes/hub_rim_back.dae" />
-            </geometry>
-        </visual>
-        <visual>
-            <origin
-                xyz="1.1934897514720447009e-14 -1.9428902930853780302e-16 0.062199999999999977529"
-                rpy="3.141592653589793116 -0 2.7052603405912831747" />
-            <geometry>
-                <mesh filename="package://zero_description/meshes/hub_rim_face.dae" />
-            </geometry>
-        </visual>
-        <visual>
             <origin
                 xyz="1.1934897514720447009e-14 -1.9428902930853780302e-16 0.027249999999999940936"
                 rpy="1.570796326794896558 -0 2.7052603405912831747" />
             <geometry>
-                <mesh filename="package://zero_description/meshes/hub_tire.dae" />
+                <mesh filename="package://zero_description/meshes/hub_wheel.dae" />
             </geometry>
         </visual>
@@ -250,5 +123,5 @@
                 rpy="1.570796326794896558 -0 2.7052603405912831747" />
             <geometry>
-                <mesh filename="package://zero_description/meshes/hub_tire.dae" />
+                <mesh filename="package://zero_description/meshes/hub_wheel.dae" />
             </geometry>
         </collision>
@@ -398,5 +271,5 @@
     <!-- ................................  PAYLOAD MODULE  .................................. -->
     <link name="payload_module">
-        <visual>
+        <collision>
             <origin
                 xyz="-1.9645968147830495471e-08 2.2406632255051934257e-07 -0.25000000000000022204"
@@ -405,5 +278,75 @@
                 <mesh filename="package://zero_description/meshes/standoff2.dae" />
             </geometry>
-        </visual>
+        </collision>
+        <visual>
+            <origin xyz="-1.9645968037643526314e-08 2.2406632246638525398e-07 -0.25" rpy="0 -0 0" />
+            <geometry>
+                <mesh filename="package://zero_description/meshes/zero_payload_system.dae" />
+            </geometry>
+        </visual>
+        <!-- Shapes for payload_system -->
+        <collision>
+            <origin xyz="0.1689999803540319645 2.2406632246638525398e-07 0.45199999999999995737"
+                rpy="-1.570796326794896558 -0 -1.57079632679489678" />
+            <geometry>
+                <box size="0.34000000000000002442 0.90400000000000002576 0.0020000000000000000416" />
+            </geometry>
+        </collision>
+        <collision>
+            <origin xyz="0.1689999803540319645 2.2406632246638525398e-07 0.45199999999999995737"
+                rpy="1.570796326794896558 -0 1.570796326794896558" />
+            <geometry>
+                <box size="0.34000000000000002442 0.90400000000000002576 0.0020000000000000000416" />
+            </geometry>
+        </collision>
+        <collision>
+            <origin xyz="-1.9645968065399101929e-08 0.16900022406632247973 0.45199999999999995737"
+                rpy="-1.570796326794896558 -0 9.2799399999999996335e-17" />
+            <geometry>
+                <box size="0.34000000000000002442 0.90400000000000002576 0.0020000000000000000416" />
+            </geometry>
+        </collision>
+        <collision>
+            <origin xyz="-0.16900001964596805815 2.2406632246638525398e-07 0.45199999999999995737"
+                rpy="-1.570796326794896558 -0 1.570796326794896558" />
+            <geometry>
+                <box size="0.34000000000000002442 0.90400000000000002576 0.0020000000000000000416" />
+            </geometry>
+        </collision>
+        <collision>
+            <origin xyz="-1.9645968009887950698e-08 -0.16899977593367751516 0.45199999999999995737"
+                rpy="-1.570796326794896558 -0 -3.141592653589793116" />
+            <geometry>
+                <box size="0.34000000000000002442 0.90400000000000002576 0.0020000000000000000416" />
+            </geometry>
+        </collision>
+        <collision>
+            <origin xyz="-0.19900001964596805704 2.2406632241087410275e-07 -0.14999999999999999445"
+                rpy="-1.570796326794896558 -0 1.5707963267948970021" />
+            <geometry>
+                <box size="0.4000000000000000222 0.2000000000000000111 0.0020000000000000000416" />
+            </geometry>
+        </collision>
+        <collision>
+            <origin xyz="-1.9645967982132375082e-08 -0.19899977593367754181 -0.14999999999999999445"
+                rpy="-1.570796326794896558 -0 -3.141592653589793116" />
+            <geometry>
+                <box size="0.4000000000000000222 0.2000000000000000111 0.0020000000000000000416" />
+            </geometry>
+        </collision>
+        <collision>
+            <origin xyz="0.19899998035403196339 2.2406632252189640522e-07 -0.14999999999999999445"
+                rpy="-1.570796326794896558 -0 -1.570796326794896336" />
+            <geometry>
+                <box size="0.4000000000000000222 0.2000000000000000111 0.0020000000000000000416" />
+            </geometry>
+        </collision>
+        <collision>
+            <origin xyz="-1.9645968093154677545e-08 0.19900022406632247862 -0.14999999999999999445"
+                rpy="-1.570796326794896558 -0 2.6124299999999998341e-16" />
+            <geometry>
+                <box size="0.4000000000000000222 0.2000000000000000111 0.0020000000000000000416" />
+            </geometry>
+        </collision>
         <collision>
             <origin
@@ -411,132 +354,15 @@
                 rpy="-1.6653345369377353037e-16 2.3453346881756870093e-17 6.0540737700961713084e-16" />
             <geometry>
-                <mesh filename="package://zero_description/meshes/standoff2.dae" />
-            </geometry>
-        </collision>
-        <visual>
-            <origin xyz="-1.9645968037643526314e-08 2.2406632246638525398e-07 -0.25" rpy="0 -0 0" />
-            <geometry>
-                <mesh filename="package://zero_description/meshes/payload_system.dae" />
-            </geometry>
-        </visual>
-        <!-- Shapes for payload_system -->
-        <collision>
-            <origin xyz="0.1689999803540319645 2.2406632246638525398e-07 0.45199999999999995737"
-                rpy="-1.570796326794896558 -0 -1.57079632679489678" />
-            <geometry>
-                <box size="0.34000000000000002442 0.90400000000000002576 0.0020000000000000000416" />
-            </geometry>
-        </collision>
-        <collision>
-            <origin xyz="0.1689999803540319645 2.2406632246638525398e-07 0.45199999999999995737"
-                rpy="1.570796326794896558 -0 1.570796326794896558" />
-            <geometry>
-                <box size="0.34000000000000002442 0.90400000000000002576 0.0020000000000000000416" />
-            </geometry>
-        </collision>
-        <collision>
-            <origin xyz="-1.9645968065399101929e-08 0.16900022406632247973 0.45199999999999995737"
-                rpy="-1.570796326794896558 -0 9.2799399999999996335e-17" />
-            <geometry>
-                <box size="0.34000000000000002442 0.90400000000000002576 0.0020000000000000000416" />
-            </geometry>
-        </collision>
-        <collision>
-            <origin xyz="-0.16900001964596805815 2.2406632246638525398e-07 0.45199999999999995737"
-                rpy="-1.570796326794896558 -0 1.570796326794896558" />
-            <geometry>
-                <box size="0.34000000000000002442 0.90400000000000002576 0.0020000000000000000416" />
-            </geometry>
-        </collision>
-        <collision>
-            <origin xyz="-1.9645968009887950698e-08 -0.16899977593367751516 0.45199999999999995737"
-                rpy="-1.570796326794896558 -0 -3.141592653589793116" />
-            <geometry>
-                <box size="0.34000000000000002442 0.90400000000000002576 0.0020000000000000000416" />
-            </geometry>
-        </collision>
-        <collision>
-            <origin xyz="-0.19900001964596805704 2.2406632241087410275e-07 -0.14999999999999999445"
-                rpy="-1.570796326794896558 -0 1.5707963267948970021" />
-            <geometry>
-                <box size="0.4000000000000000222 0.2000000000000000111 0.0020000000000000000416" />
-            </geometry>
-        </collision>
-        <collision>
-            <origin xyz="-1.9645967982132375082e-08 -0.19899977593367754181 -0.14999999999999999445"
-                rpy="-1.570796326794896558 -0 -3.141592653589793116" />
-            <geometry>
-                <box size="0.4000000000000000222 0.2000000000000000111 0.0020000000000000000416" />
-            </geometry>
-        </collision>
-        <collision>
-            <origin xyz="0.19899998035403196339 2.2406632252189640522e-07 -0.14999999999999999445"
-                rpy="-1.570796326794896558 -0 -1.570796326794896336" />
-            <geometry>
-                <box size="0.4000000000000000222 0.2000000000000000111 0.0020000000000000000416" />
-            </geometry>
-        </collision>
-        <collision>
-            <origin xyz="-1.9645968093154677545e-08 0.19900022406632247862 -0.14999999999999999445"
-                rpy="-1.570796326794896558 -0 2.6124299999999998341e-16" />
-            <geometry>
-                <box size="0.4000000000000000222 0.2000000000000000111 0.0020000000000000000416" />
-            </geometry>
-        </collision>
-        <visual>
+                <mesh filename="package://zero_description/meshes/standoff4.dae" />
+            </geometry>
+        </collision>
+        <collision>
             <origin
                 xyz="-1.9645968147830495471e-08 2.2406632255051934257e-07 -0.25000000000000022204"
                 rpy="-1.6653345369377353037e-16 2.3453346881756870093e-17 6.0540737700961713084e-16" />
             <geometry>
-                <mesh filename="package://zero_description/meshes/tray.dae" />
-            </geometry>
-        </visual>
-        <visual>
-            <origin
-                xyz="-1.9645968147830495471e-08 2.2406632255051934257e-07 -0.25000000000000022204"
-                rpy="-1.6653345369377353037e-16 2.3453346881756870093e-17 6.0540737700961713084e-16" />
-            <geometry>
-                <mesh filename="package://zero_description/meshes/standoff4.dae" />
-            </geometry>
-        </visual>
-        <collision>
-            <origin
-                xyz="-1.9645968147830495471e-08 2.2406632255051934257e-07 -0.25000000000000022204"
-                rpy="-1.6653345369377353037e-16 2.3453346881756870093e-17 6.0540737700961713084e-16" />
-            <geometry>
-                <mesh filename="package://zero_description/meshes/standoff4.dae" />
-            </geometry>
-        </collision>
-        <visual>
-            <origin
-                xyz="-1.9645968147830495471e-08 2.2406632255051934257e-07 -0.25000000000000022204"
-                rpy="-1.6653345369377353037e-16 2.3453346881756870093e-17 6.0540737700961713084e-16" />
-            <geometry>
                 <mesh filename="package://zero_description/meshes/standoff1.dae" />
             </geometry>
-        </visual>
-        <collision>
-            <origin
-                xyz="-1.9645968147830495471e-08 2.2406632255051934257e-07 -0.25000000000000022204"
-                rpy="-1.6653345369377353037e-16 2.3453346881756870093e-17 6.0540737700961713084e-16" />
-            <geometry>
-                <mesh filename="package://zero_description/meshes/standoff1.dae" />
-            </geometry>
-        </collision>
-        <visual>
-            <origin xyz="-1.0220779062274279544e-07 -0.13110197580579463494 0.77193457342055249448"
-                rpy="1.1344640137963146742 -0 5.5511151231257836882e-16" />
-            <geometry>
-                <mesh filename="package://zero_description/meshes/display.dae" />
-            </geometry>
-        </visual>
-        <visual>
-            <origin
-                xyz="-1.9645968147830495471e-08 2.2406632255051934257e-07 -0.25000000000000022204"
-                rpy="-1.6653345369377353037e-16 2.3453346881756870093e-17 6.0540737700961713084e-16" />
-            <geometry>
-                <mesh filename="package://zero_description/meshes/standoff3.dae" />
-            </geometry>
-        </visual>
+        </collision>
         <collision>
             <origin

Commit message: Added the gz_classic package

File: zero_description/urdf/zero.urdf.xacro (robot description, xacro)
@@ -45,10 +45,10 @@
     </joint>
 <!-- ................................ LIDAR .................................. -->
-    <link name="lidar"/>
-    <joint name="lidar_frame" type="fixed">
+    <link name="rplidar_laser_link"/>
+    <joint name="rplidar_laser_joint" type="fixed">
         <origin xyz="-0.00012191376555154009864 -2.8123243064170910799e-05 0.17509999999999997788"
             rpy="0 -0 0" />
         <parent link="mobile_base" />
-        <child link="lidar" />
+        <child link="rplidar_laser_link" />
         <axis xyz="0 0 0" />
     </joint>
@@ -99,5 +99,5 @@
         </inertial>
     </link>
-    <joint name="left_wheel" type="continuous">
+    <joint name="left_wheel_joint" type="continuous">
         <origin xyz="0.11279999999999962279 -1.0939515695901098363e-14 -4.7878367936959875806e-15"
             rpy="-1.570796326794896558 -0 -1.5707963267948970021" />
@@ -136,5 +136,5 @@
         </inertial>
     </link>
-    <joint name="right_wheel" type="continuous">
+    <joint name="right_wheel_joint" type="continuous">
         <origin xyz="-0.1127999999999996783 -1.09371102126810778e-14 -4.7878367936959860029e-15"
             rpy="1.570796326794896558 -0 -1.570796326794896558" />
@@ -189,5 +189,5 @@
         </inertial>
     </link>
-    <joint name="front_casterwheel" type="continuous">
+    <joint name="frontcaster_wheel_joint" type="continuous">
         <origin xyz="-0.014000000000000012434 -8.6011480390624823539e-19 0.022750000000000013267"
             rpy="-1.570796326794896558 1.570796326794896336 0" />
@@ -198,5 +198,5 @@
         <joint_properties friction="0.0" />
     </joint>
-    <joint name="front_casterpunch" type="continuous">
+    <joint name="frontcaster_rotation_joint" type="continuous">
         <origin xyz="2.2389104848756847436e-17 -0.14500000000000007327 -0.046699999999999998457"
             rpy="3.141592653589793116 -0 1.570796326794896558" />
@@ -251,5 +251,5 @@
         </inertial>
     </link>
-    <joint name="back_casterwheel" type="continuous">
+    <joint name="backcaster_wheel_joint" type="continuous">
         <origin xyz="-0.014000000000000012434 -8.601148039062451539e-19 0.022749999999999999389"
             rpy="-1.570796326794896558 -1.570796326794896336 0" />
@@ -260,5 +260,5 @@
         <joint_properties friction="0.0" />
     </joint>
-    <joint name="back_casterpunch" type="continuous">
+    <joint name="backcaster_rotation_joint" type="continuous">
         <origin xyz="-9.5525017435414730954e-17 0.14500000000000001776 -0.046699999999999998457"
             rpy="3.141592653589793116 -0 -1.570796326794896558" />
